File: O12imu.kicad_sch (KiCad schematic)
At the start: 16 parts, among them J1 Conn_01x04, J2 Conn_01x04, J3 Conn_01x06_Pin, U1 THVD1420DRLR, U2 STM32L011F4Ux, U3 LSM6DSVTR

Commit message: readme, bom, schematic pdf
Parts:
- J3: now left out of the parts list
Changed lines of the file:
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@@
   )
   (symbol (lib_id "Connector:Conn_01x06_Pin") (at 205.74 149.86 0) (mirror x) (unit 1)
-    (in_bom yes) (on_board yes) (dnp no)
+    (in_bom no) (on_board yes) (dnp no)
     (property "Reference" "J3" (at 204.47 147.32 0)
       (effects (font (size 1.27 1.27)) (justify right))
