File: O12imu.kicad_pcb (KiCad board)
At the start: 2 copper layers, 12.5 x 12.5 mm, 16 parts, among them J1 Conn_01x04, J2 Conn_01x04, J3 Conn_01x06_Pin, U1 THVD1420DRLR, U2 STM32L011F4Ux, U3 LSM6DSVTR

Commit message: shifted cap pos, readme details
Parts:
- moved C1 1.05 mm to (50.5, 44.4)
Routing:
- net GND: track 18.1 -> 19.2 mm
- net +3.3V: track 35.8 -> 34.8 mm
Changed lines of the file:
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@@
   )
   (footprint "Capacitor_SMD:C_0402_1005Metric" (layer "F.Cu")
-    (at 51.6 44.35)
+    (at 50.55 44.35)
     (descr "Capacitor SMD 0402 (1005 Metric), square (rectangular) end terminal, IPC_7351 nominal, (Body size source: IPC-SM-782 page 76, https://www.pcb-3d.com/wordpress/wp-content/uploads/ipc-sm-782a_amendment_1_and_2.pdf), generated with kicad-footprint-generator")
     (tags "capacitor")
@@
   (segment (start 50 50.9271) (end 50.499999 50.9271) (width 0.25) (layer "F.Cu") (net 4))
   (segment (start 48.8189 49.75) (end 48.8189 50) (width 0.25) (layer "F.Cu") (net 4))
-  (segment (start 52.489491 44.35) (end 52.749991 44.6105) (width 0.5) (layer "F.Cu") (net 4))
   (segment (start 48.8189 50) (end 48.8189 50.25) (width 0.25) (layer "F.Cu") (net 4))
   (segment (start 47.993395 50) (end 48.3 50) (width 0.2) (layer "F.Cu") (net 4))
@@
   (segment (start 49.75 53) (end 49.75 52.38) (width 0.25) (layer "F.Cu") (net 4))
   (segment (start 44.5 48.25) (end 44.5 47.750705) (width 0.5) (layer "F.Cu") (net 4))
+  (segment (start 52.489491 44.35) (end 52.749991 44.6105) (width 0.5) (layer "F.Cu") (net 4))
   (segment (start 49.677809 52.307809) (end 48.778416 52.307809) (width 0.25) (layer "F.Cu") (net 4))
   (segment (start 48.25 55.5) (end 47.75 55.5) (width 0.16) (layer "F.Cu") (net 4))
@@
   (segment (start 52.458211 45.6) (end 52.6555 45.797289) (width 0.2) (layer "F.Cu") (net 4))
   (segment (start 47 49.75) (end 47.743395 49.75) (width 0.2) (layer "F.Cu") (net 4))
+  (segment (start 51.03 44.35) (end 52.489491 44.35) (width 0.5) (layer "F.Cu") (net 4))
   (segment (start 50.499999 51.399999) (end 50.499999 50.9271) (width 0.25) (layer "F.Cu") (net 4))
-  (segment (start 52.08 44.35) (end 52.489491 44.35) (width 0.5) (layer "F.Cu") (net 4))
   (segment (start 44.5 51.75) (end 44.5 52.25) (width 0.5) (layer "F.Cu") (net 4))
   (segment (start 53.15 51.73) (end 52.75 51.73) (width 0.25) (layer "F.Cu") (net 4))
@@
   (segment (start 49.115 54.265) (end 48.625 53.775) (width 0.16) (layer "F.Cu") (net 6))
   (segment (start 49.5 44.67) (end 49.18 44.35) (width 0.16) (layer "F.Cu") (net 7))
-  (segment (start 49.18 44.35) (end 51.12 44.35) (width 0.5) (layer "F.Cu") (net 7))
+  (segment (start 50.07 44.35) (end 49.18 44.35) (width 0.5) (layer "F.Cu") (net 7))
   (segment (start 45.15 48.9) (end 45.15 51.28) (width 0.2) (layer "F.Cu") (net 7))
   (segment (start 45.15 51.28) (end 45.16 51.29) (width 0.2) (layer "F.Cu") (net 7))
